Commit message: s

File: description/robot_core.xacro (robot description, xacro)
@@ -13,6 +13,8 @@
     <color rgba="1.0 0.0 0.0 1.0"/>
 </material>
+<!-- BASE LINK-->
 <link name="base_link">
   </link>
+<!--CHASSIS LINK-->
 <joint name="chassis_joint" type="fixed">
     <parent link="base_link"/>
@@ -29,3 +31,32 @@
     </visual>
   </link>
+  <!--LEFT WHEEL LINK-->
+  <joint name="left_wheel_joint" type="continuous">
+    <parent link="base_link"/>
+    <child link="left wheel"/>
+    <origin xyz="0 0.175 0" rpy="-${pi/2} 0 0"/>
+    <axis xyz="0 0 1"/>
+  </joint>
+  <link name="left wheel">
+    <visual>
+      <geometry>
+        <cylinder length="0.04" radius="0.05"/>
+      </geometry>
+      <material name="black"/>
+    </visual>
+  </link>
+    <!--RIGHT WHEEL LINK-->
+    <joint name="right_wheel_joint" type="continuous">
+    <parent link="base_link"/>
+    <child link="right wheel"/>
+    <origin xyz="0 -0.175 0" rpy="${pi/2} 0 0"/>
+    <axis xyz="0 0 -1"/>
+  </joint>
+    <link name="right wheel">
+        <visual>
+        <geometry>
+            <cylinder length="0.04" radius="0.05"/>
+        </geometry>
+        <material name="red"/>
+        </visual>
 </robot>

Commit message: 1

File: description/robot_core.xacro (robot description, xacro)
@@ -24,5 +24,5 @@
 <link name="chassis">
     <visual>
-    origin xyz="0.15 0 0.75" />
+    <origin xyz="0.15 0 0.75" />
       <geometry>
         <box size="0.3 0.3 0.15"/>

Commit message: 2

File: description/robot_core.xacro (robot description, xacro)
@@ -32,31 +32,32 @@
   </link>
   <!--LEFT WHEEL LINK-->
-  <joint name="left_wheel_joint" type="continuous">
+<joint name="left_wheel_joint" type="continuous">
     <parent link="base_link"/>
     <child link="left wheel"/>
     <origin xyz="0 0.175 0" rpy="-${pi/2} 0 0"/>
     <axis xyz="0 0 1"/>
-  </joint>
-  <link name="left wheel">
+</joint>
+<link name="left wheel">
     <visual>
-      <geometry>
-        <cylinder length="0.04" radius="0.05"/>
-      </geometry>
-      <material name="black"/>
+        <geometry>
+            <cylinder length="0.04" radius="0.05"/>
+        </geometry>
+        <material name="black"/>
     </visual>
-  </link>
-    <!--RIGHT WHEEL LINK-->
-    <joint name="right_wheel_joint" type="continuous">
+</link>
+<!--RIGHT WHEEL LINK-->
+<joint name="right_wheel_joint" type="continuous">
     <parent link="base_link"/>
     <child link="right wheel"/>
     <origin xyz="0 -0.175 0" rpy="${pi/2} 0 0"/>
     <axis xyz="0 0 -1"/>
-  </joint>
-    <link name="right wheel">
-        <visual>
+</joint>
+<link name="right wheel">
+    <visual>
         <geometry>
             <cylinder length="0.04" radius="0.05"/>
         </geometry>
         <material name="red"/>
-        </visual>
+    </visual>
+<link>
 </robot>

Commit message: 1

File: description/robot_core.xacro (robot description, xacro)
@@ -15,5 +15,5 @@
 <!-- BASE LINK-->
 <link name="base_link">
-  </link>
+</link>
 <!--CHASSIS LINK-->
 <joint name="chassis_joint" type="fixed">

Commit message: 3

File: description/robot_core.xacro (robot description, xacro)
@@ -38,5 +38,5 @@
     <axis xyz="0 0 1"/>
 </joint>
-<link name="left wheel">
+<link name="left_wheel">
     <visual>
         <geometry>
@@ -53,5 +53,5 @@
     <axis xyz="0 0 -1"/>
 </joint>
-<link name="right wheel">
+<link name="right_wheel">
     <visual>
         <geometry>
@@ -60,4 +60,4 @@
         <material name="red"/>
     </visual>
-<link>
+</link>
 </robot>

Commit message: 1# Please enter the commit message for your changes. Lines starting

File: description/robot_core.xacro (robot description, xacro)
@@ -34,5 +34,5 @@
 <joint name="left_wheel_joint" type="continuous">
     <parent link="base_link"/>
-    <child link="left wheel"/>
+    <child link="left_wheel"/>
     <origin xyz="0 0.175 0" rpy="-${pi/2} 0 0"/>
     <axis xyz="0 0 1"/>
@@ -49,5 +49,5 @@
 <joint name="right_wheel_joint" type="continuous">
     <parent link="base_link"/>
-    <child link="right wheel"/>
+    <child link="right_wheel"/>
     <origin xyz="0 -0.175 0" rpy="${pi/2} 0 0"/>
     <axis xyz="0 0 -1"/>

Commit message: 1

File: description/robot_core.xacro (robot description, xacro)
@@ -24,5 +24,5 @@
 <link name="chassis">
     <visual>
-    <origin xyz="0.15 0 0.75" />
+    <origin xyz="0.15 0 0.075" />
       <geometry>
         <box size="0.3 0.3 0.15"/>

Commit message: 1

File: description/robot_core.xacro (robot description, xacro)
@@ -1,4 +1,5 @@
 <?xml version="1.0"?>
 <robot xmlns:xacro="http://www.ros.org/wiki/xacro" >
+    <xacro:include filename="inertial_macros.xacro" />
 <material name="black">
     <color rgba="0.0 0.0 0.0 1.0"/>
@@ -30,4 +31,13 @@
       <material name="white"/>
     </visual>
+    <collision>
+    <origin xyz="0.15 0 0.075" />
+      <geometry>
+        <box size="0.3 0.3 0.15"/>
+      </geometry>
+    </collision>
+    <xacro:inertial_box mass="1.0" x="0.3" y="0.3" z="0.15">
+        <origin xyz="0.15 0 0.075"/>
+    </xacro:inertial_box>
   </link>
   <!--LEFT WHEEL LINK-->
@@ -45,4 +55,12 @@
         <material name="black"/>
     </visual>
+    <collision>
+        <geometry>
+            <cylinder length="0.04" radius="0.05"/>
+        </geometry>
+    </collision>
+    <xacro:inertial_cylinder mass="0.5" length="0.04" radius="0.05">
+        <origin xyz="0 0 0"/>
+    </xacro:inertial_cylinder>
 </link>
 <!--RIGHT WHEEL LINK-->
@@ -60,4 +78,34 @@
         <material name="red"/>
     </visual>
+    <collision>
+        <geometry>
+            <cylinder length="0.04" radius="0.05"/>
+        </geometry>
+    </collision>
+    <xacro:inertial_cylinder mass="0.5" length="0.04" radius="0.05">
+        <origin xyz="0 0 0"/>
+    </xacro:inertial_cylinder>
+</link>
+<!--FRONT WHEEL LINK-->
+<joint name="front_wheel_joint" type="fixed">
+    <parent link="chassis"/>
+    <child link="front_wheel"/>
+    <origin xyz="0.15 0 0" rpy="0 0 0"/>
+</joint>
+<link name="front_wheel">
+    <visual>
+        <geometry>
+            <sphere radius="0.05"/>
+        </geometry>
+        <material name="blue"/>
+    </visual>
+    <collision>
+        <geometry>
+            <sphere radius="0.05"/>
+        </geometry>
+    </collision>
+    <xacro:inertial_sphere mass="0.5" radius="0.05">
+        <origin xyz="0 0 0"/>
+    </xacro:inertial_sphere>
 </link>
 </robot>

Commit message: 1

File: description/robot_core.xacro (robot description, xacro)
@@ -106,5 +106,5 @@
     </collision>
     <xacro:inertial_sphere mass="0.5" radius="0.05">
-        <origin xyz="0 0 0"/>
+        <origin xyz="1.5 0 0"/>
     </xacro:inertial_sphere>
 </link>

Commit message: 1

File: description/robot_core.xacro (robot description, xacro)
@@ -106,5 +106,5 @@
     </collision>
     <xacro:inertial_sphere mass="0.5" radius="0.05">
-        <origin xyz="1.5 0 0"/>
+        <origin xyz="3 0 0"/>
     </xacro:inertial_sphere>
 </link>

Commit message: 1\

File: description/robot_core.xacro (robot description, xacro)
@@ -91,5 +91,5 @@
     <parent link="chassis"/>
     <child link="front_wheel"/>
-    <origin xyz="0.15 0 0" rpy="0 0 0"/>
+    <origin xyz="0.3 0 0" rpy="0 0 0"/>
 </joint>
 <link name="front_wheel">
@@ -106,5 +106,5 @@
     </collision>
     <xacro:inertial_sphere mass="0.5" radius="0.05">
-        <origin xyz="3 0 0"/>
+        <origin xyz="0 0 0"/>
     </xacro:inertial_sphere>
 </link>

Commit message: 1

File: description/robot_core.xacro (robot description, xacro)
@@ -91,5 +91,5 @@
     <parent link="chassis"/>
     <child link="front_wheel"/>
-    <origin xyz="0.3 0 0" rpy="0 0 0"/>
+    <origin xyz="0.25 0 0" rpy="0 0 0"/>
 </joint>
 <link name="front_wheel">

Commit message: 1 1#   (use "git push" to publish your local commits)

File: description/robot_core.xacro (robot description, xacro)
@@ -91,5 +91,5 @@
     <parent link="chassis"/>
     <child link="front_wheel"/>
-    <origin xyz="0.25 0 0" rpy="0 0 0"/>
+    <origin xyz="0.22 0 0" rpy="0 0 0"/>
 </joint>
 <link name="front_wheel">

Commit message: z

File: description/robot_core.xacro (robot description, xacro)
@@ -41,4 +41,7 @@
     </xacro:inertial_box>
   </link>
+  <gazebo reference="chassis">
+    <material>Gazebo/White</material>
+    </gazebo>
   <!--LEFT WHEEL LINK-->
 <joint name="left_wheel_joint" type="continuous">
@@ -64,4 +67,7 @@
     </xacro:inertial_cylinder>
 </link>
+<gazebo reference="left_wheel">
+    <material>Gazebo/Black</material>
+</gazebo>
 <!--RIGHT WHEEL LINK-->
 <joint name="right_wheel_joint" type="continuous">
@@ -87,4 +93,7 @@
     </xacro:inertial_cylinder>
 </link>
+<gazebo reference="right wheel">
+    <material>gazebo/red<material>
+</gazebo>
 <!--FRONT WHEEL LINK-->
 <joint name="front_wheel_joint" type="fixed">
@@ -109,3 +118,6 @@
     </xacro:inertial_sphere>
 </link>
+<gazebo refenece="front_wheel">
+    <material>gazebo/blue</material>
+    </gazerbo>
 </robot>

Commit message: z

File: description/robot_core.xacro (robot description, xacro)
@@ -40,8 +40,8 @@
         <origin xyz="0.15 0 0.075"/>
     </xacro:inertial_box>
-  </link>
-  <gazebo reference="chassis">
+</link>
+<gazebo reference="chassis">
     <material>Gazebo/White</material>
-    </gazebo>
+</gazebo>
   <!--LEFT WHEEL LINK-->
 <joint name="left_wheel_joint" type="continuous">
@@ -94,5 +94,5 @@
 </link>
 <gazebo reference="right wheel">
-    <material>gazebo/red<material>
+    <material>gazebo/red</material>
 </gazebo>
 <!--FRONT WHEEL LINK-->
@@ -118,6 +118,6 @@
     </xacro:inertial_sphere>
 </link>
-<gazebo refenece="front_wheel">
+<gazebo reference="front_wheel">
     <material>gazebo/blue</material>
-    </gazerbo>
+</gazebo>
 </robot>
