Commit message: 1#

File: description/laser.xacro (robot description, xacro)
@@ -1,5 +1,5 @@
 <?xml version="1.0"?>
 <robot xmlns:xacro="http://www.ros.org/wiki/xacro"  name="robot">
-    <joint name="laser_joint" type=fixed>
+    <joint name="laser_joint" type="fixed">
         <parent link="chassis"/>
         <child link="laser_frame"/>

Commit message: 1

File: description/laser.xacro (robot description, xacro)
@@ -9,5 +9,5 @@
         <visual>
             <geometry>
-                <cylinder length="0.05" radius="0.02"/>
+                <cylinder length="0.05" radius="0.5"/>
             </geometry>
             <material name="red"/>

Commit message: 1

File: description/laser.xacro (robot description, xacro)
@@ -9,5 +9,5 @@
         <visual>
             <geometry>
-                <cylinder length="0.05" radius="0.5"/>
+                <cylinder length="0.05" radius="0.05"/>
             </geometry>
             <material name="red"/>
@@ -22,3 +22,32 @@
         </xacro:inertial_cylinder>
     </link>
+    <gazebo reference="laser_frame">
+        <sensor name="laser" type="ray">
+            <pose>0 0 0 0 0 0</pose>
+            <visual>true</visual>
+            <update_rate>10</update_rate>
+            <ray>
+                <scan>
+                    <horizontal>
+                    <samples>360</samples>
+                    <resolution>1</resolution>
+                    <min_angle>-3.14</min_angle>
+                    <max_angle>3.14</max_angle>
+                    </horizontal>
+                </scan>
+                <range>
+                    <min>0.3</min>
+                    <max>12</max>
+                    <resolution>0.01</resolution>
+                </range>
+            </ray>
+            <plugin name="laser_controller" filename="libgazebo_ros_ray_sensor.so">
+                <ros>
+                    <argument>~/out=:scan</argument>
+                </ros>
+                <output_type>sensor_msgs/LaserScan</output_type>
+                <frame_name>laser_frame</frame_name>
+            </plugin>
+        </sensor>
+    </gazebo>
 </robot>

Commit message: 1

File: description/laser.xacro (robot description, xacro)
@@ -23,4 +23,5 @@
     </link>
     <gazebo reference="laser_frame">
+        <material>Gazebo/red</material>
         <sensor name="laser" type="ray">
             <pose>0 0 0 0 0 0</pose>

Commit message: 1``

File: description/laser.xacro (robot description, xacro)
@@ -24,9 +24,11 @@
     <gazebo reference="laser_frame">
         <material>Gazebo/red</material>
-        <sensor name="laser" type="ray">
+        <sensor name="laser" type="gpu_lidar">
             <pose>0 0 0 0 0 0</pose>
-            <visual>true</visual>
+            <topic>/scan</topic>
+            <gz_frame_id>laser_frame</gz_frame_id>
+            <visualize>true</visualize>
             <update_rate>10</update_rate>
-            <ray>
+            <lidar>
                 <scan>
                     <horizontal>
@@ -42,12 +44,5 @@
                     <resolution>0.01</resolution>
                 </range>
-            </ray>
-            <plugin name="laser_controller" filename="libgazebo_ros_ray_sensor.so">
-                <ros>
-                    <argument>~/out=:scan</argument>
-                </ros>
-                <output_type>sensor_msgs/LaserScan</output_type>
-                <frame_name>laser_frame</frame_name>
-            </plugin>
+            </lidar>
         </sensor>
     </gazebo>
